Commit message: update ver 7

File: dashgo_description/urdf/dashgobase/dashgo.gazebo.xacro (robot description, xacro)
@@ -139,4 +139,5 @@
     </sensor>
   </gazebo>
+<!--
   <gazebo reference="sonar_link_fake">
     <sensor type="ray" name="TeraRanger">
@@ -176,5 +177,4 @@
    </sensor>
   </gazebo>
-  <!--link : https://www.raspberrypi.org/documentation/hardware/camera/-->
   <gazebo reference="camera_rgb_frame">
     <sensor type="camera" name="Pi Camera">
@@ -211,3 +211,4 @@
     <material>Gazebo/Black</material>
   </gazebo>
+-->
 </robot>

File: dashgo_description/urdf/dashgobase/dashgo.urdf.xacro (robot description, xacro)
@@ -202,5 +202,5 @@
   <link name="laser_frame">
     <visual>
-      <origin xyz="0 0 0.0" rpy="0 0 0"/>
+      <origin xyz="0 0 0.01" rpy="0 0 0"/>
       <geometry>
         <mesh filename="package://dashgo_description/urdf/dashgobase/meshes/sensors/laser_frame.STL"/>
